File: eagle/airu-bb.sch (EAGLE design)
At the start: 34 parts, among them IC1 DS1307, Q2 MOSFET-NCHANNELAO3404A, U1 BMP180, U2 DHT22, U3 GPS, X2 53261-08, Y1 32.768kHz

Commit message: Added modifications for AirU V2.0
This commit includes all modifications needed for AirU V2.0. This includes:

* Schematic additions integrating a mode button and real-time clock
* Board layout revisions to integrate the added components
* Changes to the BOM to reflect the new design

I also reorganized the repository structure.
Parts:
- removed R7, R8: 10k, SparkFun-Passives:RESISTOR1206
- removed SJ1: JUMPER-PAD-3-2OF3_NC_BY_TRACE_SMALL, SparkFun-Passives:JUMPER-PAD-3-2OF3_NC_BY_TRACE_SMALL
- removed Y1: 32.768kHz, SparkFun-FreqCtrl:CRYSTAL32-SMD
- added C5: 10uF, SparkFun-Passives:CAP1206
- added C6: 0.1uF, SparkFun-Passives:CAP1206
- added Y2: 32.768kHz, Lowduino:FX12232.768KHZ
Connections:
- removed net N$13: R7.2, SJ1.1
- removed net N$15: R8.2, SJ1.3
- net 5V: now also C5.2, C6.2; no longer SJ1.2
- net GND: now also C5.1, C6.1
- net N$12: now also Y2.1; no longer Y1.2
- net N$14: now also Y2.2; no longer Y1.1
- net SCL: no longer R8.1
- net SDA: no longer R7.1
Other:
- note added: "2.0"
- note removed: "1.0"
- moved on the sheet: C2
