File: eagle/airu-board.brd (EAGLE design)
At the start: 72.1 x 43.2 mm, 76 parts, among them J1 MM8030-2610RJ3, U2 HDC1080, U3 OPT3001, U5 USD-SOCKET, U6 BQ24070, X1 53261-08

Commit message: Added Step Down Converter for Power and basic layout.
Parts:
- removed C3: 0.1uF, microbuilder:_0402
- removed CN1: (no value), microbuilder:JSTPH2
- removed LED1, PWR_NPG: (no value), microbuilder:CHIPLED_1206
- removed R23: DNP, microbuilder:0402
- removed TP2, TP3: TEST-POINT2, SparkFun-Passives:PAD.02X.02
- removed U$1, U$2: U.FL, microbuilder:U.FL
- removed X1: 53261-08, con-molex:53261-08
- added C15, C16, C29: 1uF, microbuilder:_0402
- added C17: .01u, microbuilder:_0402
- added C20, C28: DNP, microbuilder:0805
- added C21: 22uF, microbuilder:0805
- added C25: 33uF, microbuilder:1206
- added C26: 1uF, microbuilder:0402
- added C27: 10uF, microbuilder:0805
- added C30: 0.1uF, microbuilder:_0402
- added GPS_FIX, PWR_PG: (no value), microbuilder:CHIPLED_1206
- added H1, H2, H3, H4: MOUNT-PAD-3.0mm, holes:3,0-PAD
- added J3: U.FL, microbuilder:U.FL
- added J4: 53261-08, con-molex:53261-08
- added J5: (no value), adafruit:USB-MINIB
- added J6: (no value), microbuilder:JSTPH2
- added JP1: (no value), jumper:JP3Q
- added L4: 10uH, laird:TYS4030*
- added Q1: (no value), adafruit:SOT23
- added R35, R50, R51: 0, microbuilder:0402
- added R38: 33, microbuilder:0402
- added R39: 330, microbuilder:0402
- added R40, R41, R44: 10k, microbuilder:0402
- added R42, R43: DNP, microbuilder:0402
- added R48: 820, microbuilder:0402
- added R49: 500k, pot:B25P
- added R53, R54: 100k, microbuilder:0402
- added R55: 270, microbuilder:0402
- added SJ1, SJ2, SJ3, SJ4: (no value), jumper:SJ
- added TP4, TP5: TEST-POINT2, SparkFun-Passives:PAD.02X.02
- added U7: BQ24070, texas:R-PVQFN-N20
- added U8: TPS54202, texas:TSOT23-6_DDC
- BAT1: device SparkFun-Electromechanical:BATTCON_20MM -> SparkFun-Electromechanical:BATTCON_12MM
- C14: value 33uF -> 0.1uF; device microbuilder:_0402 -> microbuilder:0402
- C5, C6: value 1uF -> 0.1uF
- C7: value .01u -> 0.1uF
- FB2: value 60R -> (none)
- J2: value (none) -> U.FL; device adafruit:USB-MINIB -> microbuilder:U.FL
- R11: value 330 -> 33
- R13: value 10k -> 82
- R17, R18: value 2k -> 2.7k
- R19: value 10k -> 51
- R22: value DNP -> 82
- R24: value 10k -> 100k
- R25: value 33 -> 22.1k
- R27: value 10k -> DNP
- R7: value DNP -> 500k; device microbuilder:0402 -> pot:B25P
- R8: value DNP -> 820
- R9: value 33 -> 10k
- U5: value USD-SOCKET -> MICS-4514; device SparkFun-Connectors:MICROSD_1:1 -> SparkFun-Sensors:MICS_10-SMD
- U6: value BQ24070 -> USD-SOCKET; device texas:R-PVQFN-N20 -> SparkFun-Connectors:MICROSD_1:1
- moved C4 317.3 mm to (-110.5, -336.6)
- moved R33 305.8 mm to (79.5, 21.5), turned to 90 degrees
- moved PWR_STAT2 304.3 mm to (83.0, 21.5), turned to 270 degrees
- moved R32 295.3 mm to (79.5, 18.0), turned to 270 degrees
- moved PWR_STAT1 294.0 mm to (83.0, 18.2), turned to 270 degrees
- moved R34 283.0 mm to (28.3, 26.2), turned to 180 degrees
- moved C7 278.7 mm to (-110.5, -340.4)
- moved R31 247.0 mm to (5.50, 20.5), turned to 180 degrees
- moved R26 244.0 mm to (28.5, 32.0), turned to 180 degrees
- moved R30 240.4 mm to (20.5, 11.5), turned to 180 degrees
- moved R29 239.9 mm to (23.5, 11.5)
- moved R28 237.4 mm to (20.5, 13.0), turned to 180 degrees
- moved R22 234.3 mm to (14.0, 39.0), turned to 180 degrees
- moved R13 226.6 mm to (14.0, 40.5), turned to 180 degrees
- moved R19 225.4 mm to (14.0, 31.5), turned to 180 degrees
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Connections:
- removed net CC_GPIO0: U1.P44
- removed net CC_GPIO15: U1.P6
- removed net CC_GPIO22: U1.P11
- removed net CC_GPIO28: U1.P19
- removed net CC_GPIO30: U1.P42
- removed net CC_GPIO5: U1.P50
- removed net N$6: FB2.2, J2.GND
- removed net PWR_NPG: R31.2, U6.18
- removed net USB_D+: R7.1
- removed net USB_D-: R8.1
- removed net VBAT: BAT1.1, C5.1, U4.P$4
- removed net VCC_5V: TP2.P$1, X1.8
- removed net V_OUT: C8.1, C9.1, U6.15, U6.16, U6.17
- removed net V_SYS: C3.1, C4.1, C6.1, C7.1, R10.2, R17.2, R18.2, R20.2, R21.2, R22.2, R23.2, R24.2, R34.2, U1.P36, U1.P37, U1.P40, U2.P5, U3.P1, U4.P$1, U5.4, U5.CD2
- new net MICS_PREHEAT_NOX: Q1.1, U1.P11
- new net N$21: C20.1, R24.1, R25.2, U8.4
- new net N$26: C7.1, U8.6
- new net N$29: R51.1, R8.2, U5.D
- new net N$30: J3.3, U4.P$11
- new net N$31: GPS_FIX.A, U4.P$5
- new net N$32: GPS_FIX.C, R39.2
- new net N$33: C7.2, L4.P1, U8.2
- new net N$39: FB1.1, J5.VBUS
- new net N$40: R48.2, R50.1, U5.B
- new net N$41: C20.2, C21.1, C28.1, L4.P2, R24.2, SJ4.1
- new net N$43: R7.E, R8.1
- new net N$44: R38.2, U4.P$9
- new net N$47: R48.1, R49.E
- new net N$48: JP1.1, JP1.3, JP1.5, R55.1
- new net PWR_PG: R31.2, U7.18
- new net VBAT_3V3: BAT1.PWR@1, C15.1, U4.P$4
- new net V_3V3: C14.1, C16.1, C17.1, C26.1, C29.1, C30.1, C5.1, C6.1, FB2.1, FB2.2, PWR_PG.A, PWR_STAT1.A, PWR_STAT2.A, R10.2, R17.2, R18.2, R20.2, R21.2, R34.2, R42.2, R43.2, R55.2, R9.2, SJ4.2, U1.P36, U1.P37, U1.P40, U2.P5, U3.P1, U4.P$1, U6.4, U6.CD2
- new net V_4V4: C27.1, C4.1, C8.1, C9.1, R35.1, SJ2.1, U8.3
- new net V_5V: J4.8, TP4.P$1, U5.F, U5.G, U5.H, U5.J
- new net V_OX: R50.2, U1.P48
- new net V_RED: R51.2, U1.P49
- net CC_I2C_SCL: now also R18.1, U1.P5; no longer R17.1, U1.P3
- net CC_I2C_SDA: now also R17.1; no longer R18.1
- net CC_SDCARD_CLK: now also R44.2, U6.5; no longer R27.2, U5.5
- net CC_SDCARD_CMD: now also R43.1, U6.3; no longer R23.1, U5.3
- net CC_SDCARD_DATA0: now also R42.1, U1.P6, U6.7; no longer R22.1, U1.P54, U5.7
- net CC_SOP0: now also JP1.6, R54.2
- net CC_SOP1: now also JP1.4, R53.2
- net CC_TCX0_END/SOP2: now also JP1.2
- net CC_UART0_RX: now also R38.1, U1.P10; no longer R9.2, U1.P47, U4.P$9
- net CC_UART0_TX: now also R12.2; no longer R26.2
- net CC_UART1_RX: now also R11.1, U1.P47; no longer R25.1, U1.P49
- net CC_UART1_TX: now also J4.5, R26.2; no longer R12.2, X1.5
- net GND: now also BAT1.GND, C15.2, C16.2, C17.2, C21.2, C25.2, C26.2, C27.2, C28.2, C29.2, C30.2, J2.1, J2.2, J3.1, J3.2, J4.7, J5.GND, J6.1, Q1.2, R22.1, R25.1, R27.2, R39.1, R40.1, R41.1, R44.1, R49.A, R49.S, R53.1, R54.1, R7.A, R7.S, TP5.P$1, U6.6, U6.GND1, U6.GND3, U7.11, U7.19, U7.20, U8.1; no longer BAT1.2, C3.2, C7.2, CN1.1, FB2.1, R11.1, R13.1, R27.1, TP3.P$1, U$1.1, U$1.2, U$2.1, U$2.2, U5.6, U5.GND1, U5.GND3, U6.11, U6.19, U6.20, X1.7
- net GPS_NRESET: now also R41.2, U1.P3; no longer R19.2, U1.P5
- net N$10: now also C25.1, SJ3.1, U7.5, U7.6; no longer J2.D-, R8.2
- net N$11: now also J4.4, R11.2; no longer R9.1
- net N$12: now also R27.1, R35.2, U8.5; no longer R25.2, X1.4
- net N$13: now also R13.2, U5.A; no longer LED1.A, U4.P$5
- net N$14: now also Q1.3, R13.1, R19.2; no longer LED1.C, R11.2
- net N$16: now also U7.1; no longer U6.1
- net N$17: now also U7.10; no longer U6.10
- net N$18: now also U7.13; no longer U6.13
- net N$19: now also R22.2, U5.C; no longer U$1.3, U4.P$11
- net N$20: now also U1.P9; no longer U1.P48
- net N$23: now also PWR_PG.C; no longer PWR_NPG.C
- net N$25: now also U7.14; no longer U6.14
- net N$5: now also SJ1.1, U7.4; no longer FB1.1, J2.VBUS
- net N$8: now also J2.3; no longer U$2.3
- net N$9: now also SJ2.2, U7.15, U7.16, U7.17; no longer J2.D+, R7.2
- net PM_RST: now also J4.3, R9.1, U1.P53; no longer R24.1, U1.P9, X1.3
- net PM_SET: now also J4.6, U1.P54; no longer U1.P10, X1.6
- net PWR_CE: now also U1.P50, U7.9; no longer U1.P52, U6.9
- net PWR_ISET2: now also U7.7; no longer U6.7
- net PWR_MODE: now also U1.P52, U7.8; no longer U1.P53, U6.8
- net PWR_STAT1: now also U7.2; no longer U6.2
- net PWR_STAT2: now also U7.3; no longer U6.3
- net SDCARD_CD: now also R40.2, U1.P44, U6.CD1; no longer R13.2, U5.CD1
- net VBUS_USB: now also SJ1.2; no longer PWR_NPG.A, PWR_STAT1.A, PWR_STAT2.A, U6.4
- net V_BPCK: now also J6.2, SJ3.2; no longer C14.1, CN1.2, U6.5, U6.6
Other:
- board size 72.1 x 43.2 mm -> 94 x 58.5 mm

Commit message: Finished Plexus schematic design review modifications.
This commit includes all modifications made to address the feedback
received from the engineers at Plexus. It also includes an exported
copy of all of the libraries used in the new design, which includes:
symbols, packages, and devices for each component in the schematic.
Parts:
- removed C10, C12, C7, C8: 0.1uF, microbuilder:_0402
- removed C11: 10nF, microbuilder:_0402
- removed C13, C9: 10uF, microbuilder:_0402
- removed C20, C28: DNP, microbuilder:0805
- removed C21: 22uF, microbuilder:0805
- removed C25: 33uF, microbuilder:1206
- removed C27: 10uF, microbuilder:0805
- removed PWR_PG, PWR_STAT1, PWR_STAT2: (no value), microbuilder:CHIPLED_1206
- removed R14: 1.07k, microbuilder:0402
- removed R24: 100k, microbuilder:0402
- removed R25: 22.1k, microbuilder:0402
- removed R27: DNP, microbuilder:0402
- removed R28, R30: 10k, microbuilder:0402
- removed R29, R35, R50, R51: 0, microbuilder:0402
- removed R31, R32, R33: 1.5k, microbuilder:0402
- removed R49, R7: 500k, pot:B25P
- removed SJ1, SJ2, SJ3, SJ4: (no value), jumper:SJ
- added C3: 0.1uF, microbuilder:_0402
- added CIN1, CIN3: 22uF, AcceleratedDesigns_Lib:1206_190
- added CIN2, CIN4: DNP, AcceleratedDesigns_Lib:1206_190
- added COUT1, COUT2, COUT_1, COUT_2: 22uF, AcceleratedDesigns_Lib:0805
- added CVINA1, CVINA2: 100nF, AcceleratedDesigns_Lib:0603
- added L5: 1.8uH, AcceleratedDesigns_Lib:SDR0403
- added R23: 500k, pot:B25P
- added RFBB1: 137k, AcceleratedDesigns_Lib:0402
- added RFBB2: 140k, AcceleratedDesigns_Lib:0402
- added RFBT1: 768k, AcceleratedDesigns_Lib:0402
- added RFBT2: 1.26M, AcceleratedDesigns_Lib:0805
- added U9: TLV2333, texas:DGK_S-PDSO-G8
- BAT1: value (none) -> 300TR; device SparkFun-Electromechanical:BATTCON_12MM -> airu-parts:BATTCON_12MM
- H1, H2, H3, H4: value MOUNT-PAD-3.0mm -> MOUNT-HOLE2.8; device holes:3,0-PAD -> holes:2,8
- J2, J3: value U.FL -> U.FL-R-SMT-1(10)
- J5: value (none) -> ST10S008V4BR1800; device adafruit:USB-MINIB -> SparkFun-Connectors:MICROSD_1:1
- J6: value (none) -> 47491-0001; device microbuilder:JSTPH2 -> airu-parts:USB-MINIB
- JTAG1: value (none) -> 3220-10-0100-00
- L4: value 10uH -> 1.0uH; device laird:TYS4030* -> AcceleratedDesigns_Lib:SRN3015
- Q1: value (none) -> BSS138LT3G
- R15: value 37.4k -> 10k
- R16: value 10k -> 500k; device microbuilder:0402 -> pot:B25P
- S1: value (none) -> BF3-1000
- U1: value (none) -> CC3200MODR1M2AMOBR
- U2: value HDC1080 -> HDC1080DMBT
- U3: value OPT3001 -> OPT3001DNPT
- U6: value USD-SOCKET -> ADS1015-Q1; device SparkFun-Connectors:MICROSD_1:1 -> texas:S-PDSO-G10
- U7: value BQ24070 -> TPS63020DSJR; device texas:R-PVQFN-N20 -> AcceleratedDesigns_Lib:R-PVSON-N14
- U8: value TPS54202 -> TPS63020DSJR; device texas:TSOT23-6_DDC -> AcceleratedDesigns_Lib:R-PVSON-N14
- moved C4 352.0 mm to (-1.00, -2.00)
- moved J6 86.8 mm to (3.81, 13.9)
- moved H4 85.6 mm to (90.0, 4.00)
- moved H1 85.5 mm to (4.00, 4.00)
- moved J5 70.1 mm to (73.7, 8.93), flipped to the bottom, turned to 90 degrees
- moved U6 47.5 mm to (26.0, 44.0)
- moved R15 29.3 mm to (25.0, 39.0), turned to 270 degrees
- moved JP1 27.2 mm to (89.5, 14.0), turned to 90 degrees
- moved C29 26.5 mm to (79.0, 24.0), flipped to the bottom
- moved C30 26.5 mm to (81.5, 24.0), flipped to the bottom
- moved U7 26.0 mm to (42.0, 10.5), turned to 180 degrees
- moved R16 25.2 mm to (4.00, 29.0), turned to 90 degrees
- moved J3 25.0 mm to (91.6, 30.1)
- moved R55 25.0 mm to (89.0, 19.0), turned to 180 degrees
- moved R42 24.0 mm to (72.2, 14.1), flipped to the bottom, turned to 270 degrees
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Connections:
- removed net N$23: PWR_PG.C, R31.1
- removed net N$25: R29.1, U7.14
- removed net N$26: C7.1, U8.6
- removed net N$27: PWR_STAT1.C, R32.1
- removed net N$28: PWR_STAT2.C, R33.1
- removed net N$29: R51.1, R8.2, U5.D
- removed net N$33: C7.2, L4.P1, U8.2
- removed net N$40: R48.2, R50.1, U5.B
- removed net N$41: C20.2, C21.1, C28.1, L4.P2, R24.2, SJ4.1
- removed net N$43: R7.E, R8.1
- removed net N$47: R48.1, R49.E
- removed net PWR_CE: R28.2, U1.P50, U7.9
- removed net PWR_ISET2: R16.2, U1.P51, U7.7
- removed net PWR_MODE: R30.2, U1.P52, U7.8
- removed net PWR_PG: R31.2, U7.18
- removed net PWR_STAT1: R32.2, U7.2
- removed net PWR_STAT2: R33.2, U7.3
- removed net V_4V4: C27.1, C4.1, C8.1, C9.1, R35.1, SJ2.1, U8.3
- removed net V_BPCK: J6.2, SJ3.2
- removed net V_OX: R50.2, U1.P48
- removed net V_RED: R51.2, U1.P49
- new net ADC_CONV_RDY: R15.1, U1.P49, U6.2
- new net N$24: R23.E, R8.1
- new net N$6: L5.2
- new net VOX_RAWA: R48.2, U5.B, U9.3
- new net VOX_RAWB: U6.4, U9.1, U9.2
- new net VRED_RAWA: R8.2, U5.D, U9.5
- new net VRED_RAWB: U6.5, U9.6, U9.7
- net CC_I2C_SCL: now also U6.10
- net CC_I2C_SDA: now also U6.9
- net CC_NRESET: now also U8.14
- net CC_SDCARD_CLK: now also J5.5; no longer U6.5
- net CC_SDCARD_CMD: now also J5.3; no longer U6.3
- net CC_SDCARD_DATA0: now also J5.7; no longer U6.7
- net GND: now also C3.2, CIN1.2, CIN2.2, CIN3.2, CIN4.2, COUT1.2, COUT2.2, COUT_1.2, COUT_2.2, CVINA1.2, CVINA2.2, J5.6, J5.GND1, J5.GND3, J6.GND, R16.A, R16.S, R23.A, R23.S, RFBB1.P2, RFBB2.P2, U6.1, U6.3, U7.15, U8.15, U9.4; no longer C10.2, C11.2, C12.2, C13.2, C21.2, C25.2, C27.2, C28.2, C8.2, C9.2, J5.GND, J6.1, R14.2, R15.2, R25.1, R27.2, R29.2, R49.A, R49.S, R7.A, R7.S, U6.6, U6.GND1, U6.GND3, U7.11, U7.19, U7.20, U8.1
- net N$10: now also L4.1; no longer C25.1, SJ3.1, U7.5
- net N$12: now also L4.2; no longer R27.1, R35.2, U8.5
- net N$16: now also RFBB1.P1, RFBT1.P2; no longer C10.1, U7.1
- net N$17: now also RFBB2.P1, RFBT2.2; no longer R14.1, U7.10
- net N$18: now also CVINA2.1, U7.12; no longer C11.1, R15.1, U7.13
- net N$21: now also R16.E, R48.1; no longer C20.1, R24.1, R25.2, U8.4
- net N$39: now also J6.VBUS; no longer J5.VBUS
- net N$5: now also CVINA1.1, U8.12; no longer SJ1.1, U7.4
- net N$9: now also L5.1, U8.6; no longer SJ2.2, U7.15, U7.16, U7.17
- net SDCARD_CD: now also J5.CD1; no longer U6.CD1
- net VBUS_USB: now also CIN1.1, CIN2.1, CIN3.1, CIN4.1, U7.10, U8.10; no longer C12.1, C13.1, R16.1, R28.1, R30.1, SJ1.2
- net V_3V3: now also COUT1.1, COUT_1.1, J5.4, J5.CD2, R15.2, RFBT1.P1, U8.4; no longer PWR_PG.A, PWR_STAT1.A, PWR_STAT2.A, SJ4.2, U6.4, U6.CD2
- net V_5V: now also C3.1, C4.1, COUT2.1, COUT_2.1, RFBT2.1, U6.8, U7.4, U9.8
Other:
- board size 94 x 58.5 mm -> 94 x 60 mm

Commit message: Added power and system status LEDs.
Parts:
- removed GPS_FIX: (no value), microbuilder:CHIPLED_1206
- added LED1, LED2, LED6, STAT1, STAT2, STAT3: (no value), led:CHIPLED_0603
- added PAD1, PAD2, PAD3, PAD4, PAD5: (no value), wirepad:2,54/1,0
- added R14, R24, R7: 330, microbuilder:0402
- added R25: DNP, microbuilder:0402
- added R45, R46: 330, AcceleratedDesigns_Lib:0402
- moved C4 56.0 mm to (17.0, 51.0)
- moved TP4 14.0 mm to (5.64, 56.3), flipped to the bottom
- moved JTAG1 1.00 mm to (71.3, 4.85)
- moved R10 1.00 mm to (60.0, 7.50)
- moved TP1 1.00 mm to (59.8, 10.4)
- moved J4 0.66 mm to (3.22, 50.3), flipped to the bottom, turned to 270 degrees
- moved R11 0.40 mm to (9.17, 49.3), flipped to the bottom, turned to 180 degrees
- moved R9 0.12 mm to (9.24, 51.2), flipped to the bottom, turned to 180 degrees
Connections:
- new net N$23: LED2.A, R46.P2
- new net N$25: LED1.A, R45.P2
- new net N$26: R24.1, STAT1.A
- new net N$27: R14.1, STAT2.A
- new net N$28: R7.1, STAT3.A
- new net N$29: PAD1.1, U1.P48
- new net N$33: PAD2.1, U1.P19
- new net N$34: PAD3.1, U1.P42
- new net N$35: PAD4.1, U1.P25
- new net N$36: PAD5.1, U1.P26
- new net PG_5V: R46.P1, U7.14
- new net STAT_LED1: R24.2, U1.P50
- new net STAT_LED2: R14.2, U1.P51
- new net STAT_LED3: R7.2, U1.P52
- net CC_NRESET: now also R25.2, R45.P1
- net GND: now also LED1.C, R25.1, STAT1.C, STAT2.C, STAT3.C
- net N$31: now also LED6.A; no longer GPS_FIX.A
- net N$32: now also LED6.C; no longer GPS_FIX.C
