File: eagle/airu-board.sch (EAGLE design)
At the start: 76 parts, among them J1 MM8030-2610RJ3, U2 HDC1080, U3 OPT3001, U5 USD-SOCKET, U6 BQ24070, X1 53261-08

Commit message: Added Step Down Converter for Power and basic layout.
Parts:
- removed C3: 0.1uF, microbuilder:CAP_CERAMIC_0402
- removed CN1: (no value), microbuilder:JST_2PIN
- removed LED1, PWR_NPG: (no value), microbuilder:LED1206
- removed R23: DNP, microbuilder:RESISTOR0402
- removed TP2, TP3: TEST-POINT2, SparkFun-Passives:TEST-POINT2
- removed U$1, U$2: U.FL, microbuilder:U.FL
- removed X1: 53261-08, con-molex:53261-08
- added C15, C16, C29: 1uF, microbuilder:CAP_CERAMIC_0402
- added C17: .01u, microbuilder:CAP_CERAMIC_0402
- added C20, C28: DNP, microbuilder:CAP_CERAMIC0805
- added C21: 22uF, microbuilder:CAP_CERAMIC0805
- added C25: 33uF, microbuilder:CAP_CERAMIC1206
- added C26: 1uF, microbuilder:CAP_CERAMIC0402
- added C27: 10uF, microbuilder:CAP_CERAMIC0805
- added C30: 0.1uF, microbuilder:CAP_CERAMIC_0402
- added GPS_FIX, PWR_PG: (no value), microbuilder:LED1206
- added H1, H2, H3, H4: MOUNT-PAD-3.0mm, holes:MOUNT-PAD-ROUND3.0
- added J3: U.FL, microbuilder:U.FL
- added J4: 53261-08, con-molex:53261-08
- added J5: (no value), adafruit:USBMINIB
- added J6: (no value), microbuilder:JST_2PIN
- added JP1: (no value), jumper:JP3Q
- added L4: 10uH, laird:TYS4030
- added Q1: (no value), adafruit:MOSFET-NREFLOW
- added R35, R50, R51: 0, microbuilder:RESISTOR0402
- added R38: 33, microbuilder:RESISTOR0402
- added R39: 330, microbuilder:RESISTOR0402
- added R40, R41, R44: 10k, microbuilder:RESISTOR0402
- added R42, R43: DNP, microbuilder:RESISTOR0402
- added R48: 820, microbuilder:RESISTOR0402
- added R49: 500k, pot:TRIM_US-B25P
- added R53, R54: 100k, microbuilder:RESISTOR0402
- added R55: 270, microbuilder:RESISTOR0402
- added SJ1, SJ2, SJ3, SJ4: (no value), jumper:SJ
- added TP4, TP5: TEST-POINT2, SparkFun-Passives:TEST-POINT2
- added U7: BQ24070, texas:BQ24070
- added U8: TPS54202, texas:TPS54202
- BAT1: device SparkFun-Electromechanical:BATTERY20SMD -> SparkFun-Electromechanical:BATTERY12MM
- C14: value 33uF -> 0.1uF; device microbuilder:CAP_CERAMIC_0402 -> microbuilder:CAP_CERAMIC0402
- C5, C6: value 1uF -> 0.1uF
- C7: value .01u -> 0.1uF
- FB2: value 60R -> (none)
- J2: value (none) -> U.FL; device adafruit:USBMINIB -> microbuilder:U.FL
- R11: value 330 -> 33
- R13: value 10k -> 82
- R17, R18: value 2k -> 2.7k
- R19: value 10k -> 51
- R22: value DNP -> 82
- R24: value 10k -> 100k
- R25: value 33 -> 22.1k
- R27: value 10k -> DNP
- R7: value DNP -> 500k; device microbuilder:RESISTOR0402 -> pot:TRIM_US-B25P
- R8: value DNP -> 820
- R9: value 33 -> 10k
- U5: value USD-SOCKET -> MICS-4514; device SparkFun-Connectors:USD-SOCKET -> SparkFun-Sensors:MICS-4514
- U6: value BQ24070 -> USD-SOCKET; device texas:BQ24070 -> SparkFun-Connectors:USD-SOCKET
Connections:
- removed net CC_GPIO0: U1.GPIO0
- removed net CC_GPIO15: U1.GPIO15
- removed net CC_GPIO22: U1.GPIO22
- removed net CC_GPIO28: U1.GPIO28
- removed net CC_GPIO30: U1.GPIO30
- removed net CC_GPIO5: U1.GPIO5
- removed net N$6: FB2.P$2, J2.GND
- removed net PWR_NPG: R31.2, U6.PG
- removed net USB_D+: R7.1
- removed net USB_D-: R8.1
- removed net VBAT: BAT1.+, C5.P$1, U4.VBACKUP
- removed net VCC_5V: TP2.1, X1-8.S
- removed net V_OUT: C8.P$1, C9.P$1, U6.OUT1, U6.OUT2, U6.OUT3
- removed net V_SYS: C3.P$1, C4.P$1, C6.P$1, C7.P$1, R10.2, R17.2, R18.2, R20.2, R21.2, R22.2, R23.2, R24.2, R34.2, U1.VBAT_DCDC_ANA, U1.VBAT_DCDC_DIG_IO, U1.VBAT_DCDC_PA, U2.VDD, U3.VDD, U4.VCC, U5.CD2, U5.VCC
- new net MICS_PREHEAT_NOX: Q1.G, U1.GPIO22
- new net N$21: C20.P$1, R24.1, R25.2, U8.FB
- new net N$26: C7.P$1, U8.BOOT
- new net N$29: R51.1, R8.2, U5.RS1_RED
- new net N$30: J3.SIGNAL, U4.EX_ANT
- new net N$31: GPS_FIX.A, U4.3D-FIX
- new net N$32: GPS_FIX.C, R39.2
- new net N$33: C7.P$2, L4.1, U8.SW
- new net N$39: FB1.P$1, J5.VBUS
- new net N$40: R48.2, R50.1, U5.RS1_OX
- new net N$41: C20.P$2, C21.P$1, C28.P$1, L4.2, R24.2, SJ4.1
- new net N$43: R7.E, R8.1
- new net N$44: R38.2, U4.TX
- new net N$47: R48.1, R49.E
- new net N$48: JP1.1, JP1.3, JP1.5, R55.1
- new net PWR_PG: R31.2, U7.PG
- new net VBAT_3V3: BAT1.+, C15.P$1, U4.VBACKUP
- new net V_3V3: C14.P$1, C16.P$1, C17.P$1, C26.P$1, C29.P$1, C30.P$1, C5.P$1, C6.P$1, FB2.P$1, FB2.P$2, PWR_PG.A, PWR_STAT1.A, PWR_STAT2.A, R10.2, R17.2, R18.2, R20.2, R21.2, R34.2, R42.2, R43.2, R55.2, R9.2, SJ4.2, U1.VBAT_DCDC_ANA, U1.VBAT_DCDC_DIG_IO, U1.VBAT_DCDC_PA, U2.VDD, U3.VDD, U4.VCC, U6.CD2, U6.VCC
- new net V_4V4: C27.P$1, C4.P$1, C8.P$1, C9.P$1, R35.1, SJ2.1, U8.VIN
- new net V_5V: J4-8.S, TP4.1, U5.RH2_OX, U5.RH2_RED, U5.RS2_OX, U5.RS2_RED
- new net V_OX: R50.2, U1.GPIO3
- new net V_RED: R51.2, U1.GPIO4
- net CC_I2C_SCL: now also R18.1, U1.GPIO14; no longer R17.1, U1.GPIO10
- net CC_I2C_SDA: now also R17.1; no longer R18.1
- net CC_SDCARD_CLK: now also R44.2, U6.SCK; no longer R27.2, U5.SCK
- net CC_SDCARD_CMD: now also R43.1, U6.DI; no longer R23.1, U5.DI
- net CC_SDCARD_DATA0: now also R42.1, U1.GPIO15, U6.DO; no longer R22.1, U1.GPIO9, U5.DO
- net CC_SOP0: now also JP1.6, R54.2
- net CC_SOP1: now also JP1.4, R53.2
- net CC_TCX0_END/SOP2: now also JP1.2
- net CC_UART0_RX: now also R38.1, U1.GPIO13; no longer R9.2, U1.GPIO2, U4.TX
- net CC_UART0_TX: now also R12.2; no longer R26.2
- net CC_UART1_RX: now also R11.1, U1.GPIO2; no longer R25.1, U1.GPIO4
- net CC_UART1_TX: now also J4-5.S, R26.2; no longer R12.2, X1-5.S
- net GND: now also C15.P$2, C16.P$2, C17.P$2, C21.P$2, C25.P$2, C26.P$2, C27.P$2, C28.P$2, C29.P$2, C30.P$2, J2.GND@0, J2.GND@1, J3.GND@0, J3.GND@1, J4-7.S, J5.GND, J6.1, Q1.S, R22.1, R25.1, R27.2, R39.1, R40.1, R41.1, R44.1, R49.A, R49.S, R53.1, R54.1, R7.A, R7.S, TP5.1, U6.GND, U6.SHIELD@1, U6.SHIELD@3, U7.GND1, U7.GND2, U7.VSS, U8.GND; no longer C3.P$2, C7.P$2, CN1.1, FB2.P$1, R11.1, R13.1, R27.1, TP3.1, U$1.GND@0, U$1.GND@1, U$2.GND@0, U$2.GND@1, U5.GND, U5.SHIELD@1, U5.SHIELD@3, U6.GND1, U6.GND2, U6.VSS, X1-7.S
- net GPS_NRESET: now also R41.2, U1.GPIO10; no longer R19.2, U1.GPIO14
- net N$10: now also C25.P$1, SJ3.1, U7.BAT1, U7.BAT2; no longer J2.D-, R8.2
- net N$11: now also J4-4.S, R11.2; no longer R9.1
- net N$12: now also R27.1, R35.2, U8.EN; no longer R25.2, X1-4.S
- net N$13: now also R13.2, U5.RH1_OX; no longer LED1.A, U4.3D-FIX
- net N$14: now also Q1.D, R13.1, R19.2; no longer LED1.C, R11.2
- net N$16: now also U7.VREF; no longer U6.VREF
- net N$17: now also U7.ISET1; no longer U6.ISET1
- net N$18: now also U7.DPPM; no longer U6.DPPM
- net N$19: now also R22.2, U5.RH1_RED; no longer U$1.SIGNAL, U4.EX_ANT
- net N$20: now also U1.GPIO12; no longer U1.GPIO3
- net N$23: now also PWR_PG.C; no longer PWR_NPG.C
- net N$25: now also U7.TMR; no longer U6.TMR
- net N$5: now also SJ1.1, U7.IN; no longer FB1.P$1, J2.VBUS
- net N$8: now also J2.SIGNAL; no longer U$2.SIGNAL
- net N$9: now also SJ2.2, U7.OUT1, U7.OUT2, U7.OUT3; no longer J2.D+, R7.2
- net PM_RST: now also J4-3.S, R9.1, U1.GPIO8; no longer R24.1, U1.GPIO12, X1-3.S
- net PM_SET: now also J4-6.S, U1.GPIO9; no longer U1.GPIO13, X1-6.S
- net PWR_CE: now also U1.GPIO5, U7.CE; no longer U1.GPIO7, U6.CE
- net PWR_ISET2: now also U7.ISET2; no longer U6.ISET2
- net PWR_MODE: now also U1.GPIO7, U7.MODE; no longer U1.GPIO8, U6.MODE
- net PWR_STAT1: now also U7.STAT1; no longer U6.STAT1
- net PWR_STAT2: now also U7.STAT2; no longer U6.STAT2
- net SDCARD_CD: now also R40.2, U1.GPIO0, U6.CD1; no longer R13.2, U5.CD1
- net VBUS_USB: now also SJ1.2; no longer PWR_NPG.A, PWR_STAT1.A, PWR_STAT2.A, U6.IN
- net V_BPCK: now also J6.2, SJ3.2; no longer C14.P$1, CN1.2, U6.BAT1, U6.BAT2
Other:
- note added: "1.0"
- note added: "3.3V from buck"
- note added: "4.4V -> 3.3V Step Down Converter"
- note added: "Ambient Light Sensor"
- note added: "CO/NO2 Sensor"
- note added: "GPS + RTC Module"
- note added: "Li-Ion Charger and System Power Management"
- note added: "MCU + WiFi Module"
- note added: "MCU + Wireless RF"
- note added: "PG = STAT1/2 = OFF indicates the OD transistor is off"
- note added: "PM Sensor Pin Housing"
- note added: "Power Management"
- note added: "RF Antenna Circuit"
- note added: "Sense On Power Setting Circuit"
- note added: "System Power Status LEDs"
- note added: "Temp + Humidity Sensor"
- note added: "microSD Card Connector"
- note removed: "(5V from boost converter)"
- note removed: "3.3V from LDO"
- note removed: "NPG = STAT1/2 = OFF indicates the OD transistor is off"
- note removed: "V_OUT = 4.4 V"

Commit message: Finished Plexus schematic design review modifications.
This commit includes all modifications made to address the feedback
received from the engineers at Plexus. It also includes an exported
copy of all of the libraries used in the new design, which includes:
symbols, packages, and devices for each component in the schematic.
Parts:
- removed C10, C12, C7, C8: 0.1uF, microbuilder:CAP_CERAMIC_0402
- removed C11: 10nF, microbuilder:CAP_CERAMIC_0402
- removed C13, C9: 10uF, microbuilder:CAP_CERAMIC_0402
- removed C20, C28: DNP, microbuilder:CAP_CERAMIC0805
- removed C21: 22uF, microbuilder:CAP_CERAMIC0805
- removed C25: 33uF, microbuilder:CAP_CERAMIC1206
- removed C27: 10uF, microbuilder:CAP_CERAMIC0805
- removed PWR_PG, PWR_STAT1, PWR_STAT2: (no value), microbuilder:LED1206
- removed R14: 1.07k, microbuilder:RESISTOR0402
- removed R24: 100k, microbuilder:RESISTOR0402
- removed R25: 22.1k, microbuilder:RESISTOR0402
- removed R27: DNP, microbuilder:RESISTOR0402
- removed R28, R30: 10k, microbuilder:RESISTOR0402
- removed R29, R35, R50, R51: 0, microbuilder:RESISTOR0402
- removed R31, R32, R33: 1.5k, microbuilder:RESISTOR0402
- removed R49, R7: 500k, pot:TRIM_US-B25P
- removed SJ1, SJ2, SJ3, SJ4: (no value), jumper:SJ
- added C3: 0.1uF, microbuilder:CAP_CERAMIC_0402
- added CIN1, CIN3: 22uF, AcceleratedDesigns_Lib:GRM31CR61A226KE19L
- added CIN2, CIN4: DNP, AcceleratedDesigns_Lib:GRM31CR61A226KE19L
- added COUT1, COUT2, COUT_1, COUT_2: 22uF, AcceleratedDesigns_Lib:GRM21BR60J226ME39L
- added CVINA1, CVINA2: 100nF, AcceleratedDesigns_Lib:C0603C104K8RACTU
- added L5: 1.8uH, AcceleratedDesigns_Lib:SDR0403-1R8ML
- added R23: 500k, pot:TRIM_US-B25P
- added RFBB1: 137k, AcceleratedDesigns_Lib:CRCW0402137KFKED
- added RFBB2: 140k, AcceleratedDesigns_Lib:CRCW0402137KFKED
- added RFBT1: 768k, AcceleratedDesigns_Lib:CRCW0402768KFKED
- added RFBT2: 1.26M, AcceleratedDesigns_Lib:RT0805BRD071M26L
- added U9: TLV2333, texas:TLV2333
- BAT1: value (none) -> 300TR; device SparkFun-Electromechanical:BATTERY12MM -> airu-parts:BATTERY12MM; MANUFACTURER_NAME (none) -> Keystone; MANUFACTURER_PART_NUMBER (none) -> 300TR
- H1, H2, H3, H4: value MOUNT-PAD-3.0mm -> MOUNT-HOLE2.8; device holes:MOUNT-PAD-ROUND3.0 -> holes:MOUNT-HOLE2.8
- J2, J3: value U.FL -> U.FL-R-SMT-1(10)
- J5: value (none) -> ST10S008V4BR1800; device adafruit:USBMINIB -> SparkFun-Connectors:USD-SOCKET; MANUFACTURER_NAME (none) -> JAE; MANUFACTURER_PART_NUMBER (none) -> ST10S008V4BR1800
- J6: value (none) -> 47491-0001; device microbuilder:JST_2PIN -> airu-parts:USBMINIB; MANUFACTURER_NAME (none) -> Molex; MANUFACTURER_PART_NUMBER (none) -> 47491-0001
- JTAG1: value (none) -> 3220-10-0100-00; MANUFACTURER_NAME (none) -> CNC Tech; MANUFACTURER_PART_NUMBER (none) -> 3220-10-0100-00
- L4: value 10uH -> 1.0uH; device laird:TYS4030 -> AcceleratedDesigns_Lib:SRN3015-1R0Y
- Q1: value (none) -> BSS138LT3G
- R15: value 37.4k -> 10k
- R16: value 10k -> 500k; device microbuilder:RESISTOR0402 -> pot:TRIM_US-B25P
- S1: value (none) -> BF3-1000
- U1: value (none) -> CC3200MODR1M2AMOBR
- U2: value HDC1080 -> HDC1080DMBT
- U3: value OPT3001 -> OPT3001DNPT
- U6: value USD-SOCKET -> ADS1015-Q1; device SparkFun-Connectors:USD-SOCKET -> texas:ADS1015
- U7: value BQ24070 -> TPS63020DSJR; device texas:BQ24070 -> AcceleratedDesigns_Lib:TPS63020DSJR
- U8: value TPS54202 -> TPS63020DSJR; device texas:TPS54202 -> AcceleratedDesigns_Lib:TPS63020DSJR
Connections:
- removed net N$23: PWR_PG.C, R31.1
- removed net N$25: R29.1, U7.TMR
- removed net N$26: C7.P$1, U8.BOOT
- removed net N$27: PWR_STAT1.C, R32.1
- removed net N$28: PWR_STAT2.C, R33.1
- removed net N$29: R51.1, R8.2, U5.RS1_RED
- removed net N$33: C7.P$2, L4.1, U8.SW
- removed net N$40: R48.2, R50.1, U5.RS1_OX
- removed net N$41: C20.P$2, C21.P$1, C28.P$1, L4.2, R24.2, SJ4.1
- removed net N$43: R7.E, R8.1
- removed net N$47: R48.1, R49.E
- removed net PWR_CE: R28.2, U1.GPIO5, U7.CE
- removed net PWR_ISET2: R16.2, U1.GPIO6, U7.ISET2
- removed net PWR_MODE: R30.2, U1.GPIO7, U7.MODE
- removed net PWR_PG: R31.2, U7.PG
- removed net PWR_STAT1: R32.2, U7.STAT1
- removed net PWR_STAT2: R33.2, U7.STAT2
- removed net V_4V4: C27.P$1, C4.P$1, C8.P$1, C9.P$1, R35.1, SJ2.1, U8.VIN
- removed net V_BPCK: J6.2, SJ3.2
- removed net V_OX: R50.2, U1.GPIO3
- removed net V_RED: R51.2, U1.GPIO4
- new net ADC_CONV_RDY: R15.1, U1.GPIO4, U6.ALERT
- new net N$24: R23.E, R8.1
- new net N$6: L5.2
- new net VOX_RAWA: R48.2, U5.RS1_OX, U9G$1.+
- new net VOX_RAWB: U6.AIN0, U9G$1.-, U9G$1.OUT
- new net VRED_RAWA: R8.2, U5.RS1_RED, U9G$1.+1
- new net VRED_RAWB: U6.AIN1, U9G$1.-1, U9G$1.OUT1
- net CC_I2C_SCL: now also U6.SCL
- net CC_I2C_SDA: now also U6.SDA
- net CC_NRESET: now also U8.PG
- net CC_SDCARD_CLK: now also J5.SCK; no longer U6.SCK
- net CC_SDCARD_CMD: now also J5.DI; no longer U6.DI
- net CC_SDCARD_DATA0: now also J5.DO; no longer U6.DO
- net GND: now also C3.P$2, CIN1.2, CIN2.2, CIN3.2, CIN4.2, COUT1.2, COUT2.2, COUT_1.2, COUT_2.2, CVINA1.2, CVINA2.2, J5.SHIELD@1, J5.SHIELD@3, J6.GND, R16.A, R16.S, R23.A, R23.S, RFBB1.2, RFBB2.2, U6.ADDR, U7.GND_2, U8.GND_2, U9G$2.V-; no longer C10.P$2, C11.P$2, C12.P$2, C13.P$2, C21.P$2, C25.P$2, C27.P$2, C28.P$2, C8.P$2, C9.P$2, J6.1, R14.2, R15.2, R25.1, R27.2, R29.2, R49.A, R49.S, R7.A, R7.S, U6.SHIELD@1, U6.SHIELD@3, U7.GND1, U7.GND2, U7.VSS, U8.GND
- net N$10: now also L4.1, U7.L2_2; no longer C25.P$1, SJ3.1, U7.BAT1, U7.BAT2
- net N$12: now also L4.2; no longer R27.1, R35.2, U8.EN
- net N$16: now also RFBB1.1, RFBT1.2; no longer C10.P$1, U7.VREF
- net N$17: now also RFBB2.1, RFBT2.2; no longer R14.1, U7.ISET1
- net N$18: now also CVINA2.1, U7.EN; no longer C11.P$1, R15.1, U7.DPPM
- net N$21: now also R16.E, R48.1; no longer C20.P$1, R24.1, R25.2, U8.FB
- net N$39: now also J6.VBUS; no longer J5.VBUS
- net N$5: now also CVINA1.1, U8.EN; no longer SJ1.1, U7.IN
- net N$9: now also L5.1, U8.L2_2; no longer SJ2.2, U7.OUT1, U7.OUT2, U7.OUT3
- net SDCARD_CD: now also J5.CD1; no longer U6.CD1
- net VBUS_USB: now also CIN1.1, CIN2.1, CIN3.1, CIN4.1, U7.VIN_2, U8.VIN_2; no longer C12.P$1, C13.P$1, R16.1, R28.1, R30.1, SJ1.2
- net V_3V3: now also COUT1.1, COUT_1.1, J5.CD2, J5.VCC, R15.2, RFBT1.1, U8.VOUT_2; no longer PWR_PG.A, PWR_STAT1.A, PWR_STAT2.A, SJ4.2, U6.CD2, U6.VCC
- net V_5V: now also C3.P$1, C4.P$1, COUT2.1, COUT_2.1, RFBT2.1, U6.VDD, U7.VOUT_2, U9G$2.V+
Other:
- note added: "12-bit ADC for Gas Sensors"
- note added: "Analog Buffers"
- note added: "Power Management (Buck/Boost)"
- note added: "VBUS_USB = 4.4-5.3V"
- note added: "mini-USB input"
- note removed: "(JST for Li-Ion Battery Pack)"
- note removed: "4.4V -> 3.3V Step Down Converter"
- note removed: "ICHG = 1A VDDPM-SET = 3.7V VDDPM-REG = 4.26V"
- note removed: "Li-Ion Charger and System Power Management"
- note removed: "PG = STAT1/2 = OFF indicates the OD transistor is off"
- note removed: "STAT1, STAT2, STATUS ON ON Precharge ON OFF Fast charge OFF ON Charge done OFF OFF FAULT"
- note removed: "System Power Status LEDs"
- note removed: "VBUS_USB = 5V +/- 0.1V"

Commit message: Added power and system status LEDs.
Parts:
- removed GPS_FIX: (no value), microbuilder:LED1206
- added LED1, LED2, LED6, STAT1, STAT2, STAT3: (no value), led:LEDCHIPLED_0603
- added PAD1, PAD2, PAD3, PAD4, PAD5: (no value), wirepad:2,54/1,0
- added R14, R24, R7: 330, microbuilder:RESISTOR0402
- added R25: DNP, microbuilder:RESISTOR0402
- added R45, R46: 330, AcceleratedDesigns_Lib:CRCW0402137KFKED
Connections:
- new net N$23: LED2.A, R46.2
- new net N$25: LED1.A, R45.2
- new net N$26: R24.1, STAT1.A
- new net N$27: R14.1, STAT2.A
- new net N$28: R7.1, STAT3.A
- new net N$29: PAD1.P, U1.GPIO3
- new net N$33: PAD2.P, U1.GPIO28
- new net N$34: PAD3.P, U1.GPIO30
- new net N$35: PAD4.P, U1.ANT_SEL_1
- new net N$36: PAD5.P, U1.ANT_SEL_2
- new net PG_5V: R46.1, U7.PG
- new net STAT_LED1: R24.2, U1.GPIO5
- new net STAT_LED2: R14.2, U1.GPIO6
- new net STAT_LED3: R7.2, U1.GPIO7
- net CC_NRESET: now also R25.2, R45.1
- net GND: now also LED1.C, R25.1, STAT1.C, STAT2.C, STAT3.C
- net N$31: now also LED6.A; no longer GPS_FIX.A
- net N$32: now also LED6.C; no longer GPS_FIX.C
